File: smd_breadboard.kicad_pcb (KiCad board)
At the start: 2 copper layers, 5 parts, among them J1 USB_C_Receptacle_USB2.0_14P, U1 SHT30-DIS, U2 TPL5010, U4 W25Q128JVS, U5 FT230XS

Commit message: plotted gerbers
Parts:
- added ?: , , F.Cu at (174.0, 71.1)
- added ?: , , F.Cu at (127.0, 63.5)
- added ?: , , F.Cu at (132.2, 76.2)
- added ?: , , F.Cu at (170.2, 71.1)
- added ?: , , F.Cu at (149.9, 68.6)
- added ?: , , F.Cu at (170.2, 68.6)
- added ?: , , F.Cu at (150.0, 76.2)
- added ?: , , F.Cu at (154.9, 71.1)
- added ?: , , F.Cu at (170.2, 76.2)
- added ?: , , F.Cu at (189.2, 63.5)
- added ?: , , F.Cu at (132.2, 78.7)
- added ?: , , F.Cu at (132.2, 73.7)
- added ?: , , F.Cu at (170.2, 63.5)
- added ?: , , F.Cu at (111.8, 78.7)
- added ?: , , F.Cu at (154.9, 81.3)
- added ?: , , F.Cu at (127.0, 66.0)
- added ?: , , F.Cu at (154.9, 63.5)
- added ?: , , F.Cu at (149.9, 66.0)
- added ?: , , F.Cu at (174.0, 63.5)
- added ?: , , F.Cu at (150.0, 78.7)
- added ?: , , F.Cu at (111.8, 68.6)
- added ?: , , F.Cu at (170.2, 81.3)
- added ?: , , F.Cu at (132.1, 66.0)
- added ?: , , F.Cu at (174.0, 68.6)
- added ?: , , F.Cu at (132.2, 71.1)
- added ?: , , F.Cu at (149.9, 71.1)
- added ?: , , F.Cu at (111.8, 81.3)
- added ?: , , F.Cu at (170.2, 66.0)
- added ?: , , F.Cu at (111.8, 63.5)
- added ?: , , F.Cu at (127.0, 71.1)
- added ?: , , F.Cu at (189.2, 73.7)
- added ?: , , F.Cu at (127.0, 68.6)
- added ?: , , F.Cu at (132.2, 68.6)
- added ?: , , F.Cu at (189.2, 66.0)
- added ?: , , F.Cu at (127.0, 76.2)
- added ?: , , F.Cu at (127.0, 78.7)
- added ?: , , F.Cu at (189.2, 68.6)
- added ?: , , F.Cu at (174.0, 73.7)
- added ?: , , F.Cu at (111.8, 66.0)
- added ?: , , F.Cu at (174.0, 66.0)
- added ?: , , F.Cu at (150.0, 73.7)
- added ?: , , F.Cu at (170.2, 78.7)
- added ?: , , F.Cu at (154.9, 68.6)
- added ?: , , F.Cu at (189.2, 71.1)
- added ?: , , F.Cu at (111.8, 73.7)
- added ?: , , F.Cu at (127.0, 73.7)
- added ?: , , F.Cu at (127.0, 81.3)
- added ?: , , F.Cu at (111.8, 76.2)
- added ?: , , F.Cu at (111.8, 71.1)
- added ?: , , F.Cu at (154.9, 78.7)
- added ?: , , F.Cu at (154.9, 76.2)
- added ?: , , F.Cu at (154.9, 66.0)
- QUAD 8SOIC: renamed from U4
- moved TSOT23-6 26.0 mm to (162.1, 78.4)
- moved SHT30-DIS-B2.5KS 24.5 mm to (181.3, 67.4)
- moved USB4105-GF-A 15.4 mm to (141.1, 75.1)
- moved QUAD 8SOIC 15.2 mm to (162.3, 67.5)
- moved 16SSOP 4.72 mm to (119.5, 72.3)
- renumbered U5 to 16SSOP, U1 to SHT30-DIS-B2.5KS, U2 to TSOT23-6, J1 to USB4105-GF-A
Routing:
- net (no net): track 0.00 -> 427.3 mm
Other:
- board outline added: 80 x 21.6 mm
- board text added: "CES @ KIT"
